File: schematic/schematic.sch (EAGLE design)
At the start: 6 parts, among them U1 ARDUINOR3-DIMENSION

Commit message: updated schematic
Connections:
- removed net N$12 (its old number): U$3.SIG, U1.D4
- new net N$14: U$3.SIG, U1.D0
- net N$13: now also U$4.GND; no longer BAT.-, U$3.NC
- net N$16: now also BAT.-; no longer U$4.GND
- net N$3: now also U$2.VDD
- net N$9: now also U1.D2; no longer U1.D3
