File: hardware/top_schematic.sch (EAGLE design)
At the start: 7 parts, among them U1 ARDUINOR3-DIMENSION

Commit message: improved android app, added heat index, took pictures
Parts:
- removed BAT: 1V60R, battery:1V60R
- added 9V: 1V60R, battery:1V60R
- added CX1: (no value), rcl:CXXC10B5
- added U$5: TI_LM2825, BLE_sensor_pack_parts:TI_LM2825
Connections:
- removed net VIN: BAT.+, U1.VIN
- new net N$1: 9V.+, U$5.IN@19
- new net N$15: CX1.1, U$5.SOFT@13, U$5.SOFT@14
- net N$16: now also 9V.-, CX1.2, U$5.GND@1, U$5.GND@11, U$5.GND@12, U$5.GND@2, U$5.GND@23; no longer BAT.-
- net VDD: now also U$5.OUT@5

Commit message: updated soft-start capacitor to include value in schematic
Parts:
- C1: value (none) -> 0.1uF
- renumbered CX1 to C1
Changed lines of the file:
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@@
 <part name="U$4" library="BLE_sensor_parts" deviceset="ADAFRUIT_SI1145_BREAKOUT" device=""/>
 <part name="U$5" library="BLE_sensor_pack_parts" deviceset="TI_LM2825" device=""/>
-<part name="CX1" library="rcl" deviceset="CX" device="XC10B5"/>
+<part name="C1" library="rcl" deviceset="CX" device="XC10B5" value="0.1uF"/>
 </parts>
 <sheets>
@@
 <instance part="U$4" gate="G$1" x="88.9" y="38.1"/>
 <instance part="U$5" gate="G$1" x="33.02" y="40.64"/>
-<instance part="CX1" gate="G$1" x="53.34" y="17.78"/>
+<instance part="C1" gate="G$1" x="53.34" y="17.78"/>
 </instances>
 <busses>
@@
 <wire x1="53.34" y1="50.8" x2="53.34" y2="60.96" width="0.1524" layer="91"/>
 <junction x="53.34" y="60.96"/>
-<pinref part="CX1" gate="G$1" pin="2"/>
+<pinref part="C1" gate="G$1" pin="2"/>
 <wire x1="53.34" y1="12.7" x2="53.34" y2="10.16" width="0.1524" layer="91"/>
 <wire x1="53.34" y1="10.16" x2="63.5" y2="10.16" width="0.1524" layer="91"/>
@@
 <net name="N$15" class="0">
 <segment>
-<pinref part="CX1" gate="G$1" pin="1"/>
+<pinref part="C1" gate="G$1" pin="1"/>
 <wire x1="53.34" y1="20.32" x2="53.34" y2="25.4" width="0.1524" layer="91"/>
 <pinref part="U$5" gate="G$1" pin="SOFT@14"/>
